File: anavi-wb3s-breadboard.kicad_pcb (KiCad board)
At the start: 2 copper layers, 49.5 x 19 mm, 4 parts, among them J1 Conn_01x11_Male, J2 Conn_01x11_Male, U1 ESP-12E

Commit message: anavi-wb3s-breadboard.kicad_pcb: Adjust
Adjust configurations for exporting gerber and drill files.

Signed-off-by: Leon Anavi <leon@anavi.org>
Other:
- board text removed: "Breakout Board for ESP-12E/F"
Changed lines of the file:
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@@
 			(at 0.49 -0.8 90)
 			(layer "F.Fab")
+			(hide yes)
 			(effects
 				(font
@@
 		)
 	)
-	(gr_text "Breakout Board\nfor ESP-12E/F"
-		(at 86.36 82.55 90)
-		(layer "B.SilkS")
-		(effects
-			(font
-				(size 1 1)
-				(thickness 0.15)
-			)
-			(justify mirror)
-		)
-	)

Commit message: Improve silkscreen labels
Improve the silkscreen labels and an URL.

Signed-off-by: Leon Anavi <leon@anavi.org>
Other:
- board text added: "https://anavi.technology/"
Changed lines of the file:
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@@
 			(drillshape 0)
 			(scaleselection 1)
-			(outputdirectory "fab/")
+			(outputdirectory "plots/10")
 		)
 	)
@@
 			)
 			(justify left bottom mirror)
+		)
+	)
+	(gr_text "https://anavi.technology/"
+		(at 110.5 91 0)
+		(layer "B.SilkS")
+		(effects
+			(font
+				(size 1 1)
+				(thickness 0.1)
+			)
+			(justify left bottom mirror)
